File: Frketic_ptp_project1/Frketic_ptp_project1.kicad_sch (KiCad schematic)
At the start: 24 parts, among them J1 Screw_Terminal_01x02, SW1 SW1, SW2 SW_SPDT_312, U1 NE555P, U2 LM2574N-5

Commit message: LV3
Parts:
- added U6: ~, Library:SOT-23-6, symbol SOT-23-6:SN74LVC1G11
Connections:
- net +5V: now also U6.5 (VCC)
- net Q1: now also U6.1 (A)
- net Q3: now also U6.3 (B)
- new net CLOCK: U6.6 (C)
- new net RESET: U6.4 (Y)
Other:
- note added: "LED diode"
- note added: "Napajanje"
- note added: "Tipkallo i ulaz radnog takta"

Commit message: erc
Parts:
- added H1, H2, H3, H4: MountingHole, symbol Mechanical:MountingHole
- added R10, R11, R12, R20, R5: 10k, symbol Device:R
- added R14, R16, R17, R18, R5, R6, R8: 2k, symbol Device:R_Small
- added U3, U4, U5: 4027, symbol 4xxx:4027
- added U7: 74LS47, symbol 74xx:74LS47
- added U8: FYS-3911BUHR-21, Display_7Segment:HDSP-7401, symbol Display_Character:HDSP-7401
- C1: footprint (none) -> Capacitor_THT:CP_Radial_D5.0mm_P2.00mm; Manufacturer (none) -> AISHI; Pat Nuber (none) -> EWH1EM220D11OT
- C2: value C_Polarized -> 220u; footprint (none) -> Capacitor_THT:CP_Radial_D5.0mm_P2.00mm; Part Number (none) -> RD1A227M05011BB; manufacturer (none) -> SAMWHA
- C4: value C4 -> 1u; footprint (none) -> Capacitor_SMD:C_1206_3216Metric_Pad1.33x1.80mm_HandSolder; Manufacturer (none) -> Capacitor_SMD:C_1206_3216Metric_Pad1.33x1.80mm_HandSolder; Part Number (none) -> CL31B105KBHNNNE
- D1: footprint (none) -> Package_DIP:DIP-8_W7.62mm_Socket_LongPads; Part Number (none) -> LM2574N-5G; manuacturer (none) -> ONSEMI
- J1: footprint (none) -> TerminalBlock_MetzConnect:TerminalBlock_MetzConnect_Type011_RT05502HBLC_1x02_P5.00mm_Horizontal; Manufacurer (none) -> DEGSON ELECTRONICS; Part Number (none) -> DG301-5.0-02P-12-00A(H)
- R13: renamed from R2; value R2 -> 2k; footprint (none) -> Resistor_SMD:R_1206_3216Metric_Pad1.30x1.75mm_HandSolder; Manufacturer (none) -> ROYALOHM; Part Number (none) -> 1206S4F2001T5E
- R7: renamed from R1; value 2k -> 10k; footprint (none) -> Resistor_SMD:R_1206_3216Metric_Pad1.30x1.75mm_HandSolder
- SW1: footprint (none) -> Button_Switch_THT:SW_PUSH_6mm_H4.3mm; Manufactuer (none) -> microswitch TACT; Par Number (none) -> TACT-64N-F
- SW2: footprint (none) -> Button_Switch_THT:SW_Slide_SPDT_Straight_CK_OS102011MS2Q; Manufactuer (none) -> C&K; Part Number (none) -> OS102011MS2QN1C
- U2: footprint Package_DIP:DIP-8_W7.62mm -> Package_DIP:DIP-8_W7.62mm_Socket_LongPads; Manufacturer (none) -> ONSEMI; Part Nube (none) -> LM2574N-5G
Connections:
- net Clock is gone; now on net CLOCK: SW2.1 (B)
- net +5V: now also R10.1, R11.1, R12.1, R20.1, R5.1, U3.16 (VDD), U4.16 (VDD), U7.16 (VCC), U8.1 (CA), U8.6 (CA)
- net CLOCK: now also U3.3 (C)
- net GND: now also U3.7 (S), U3.8 (VSS), U3.9 (S), U4.8 (VSS), U4.9 (S), U5.9 (S), U7.8 (GND)
- net Q0: now also U3.1 (Q), U3.13 (C), U7.7 (A)
- net Q1: now also U3.15 (Q), U4.13 (C), U7.1 (B)
- net Q2: now also U4.15 (Q), U5.13 (C), U7.2 (C)
- net Q3: now also U5.15 (Q), U7.6 (D)
- new net: R12.2, U5.10 (J), U5.11 (K)
- new net: R5.2, U3.5 (K), U3.6 (J)
- new net: R16.1, U7.9 (e)
- new net: R16.2, U8.4 (E)
- new net: R14.1, U7.10 (d)
- new net: R14.2, U8.5 (D)
- new net: R11.2, U4.10 (J), U4.11 (K)
- new net: R5.1, U7.13 (a)
- new net: R5.2, U8.10 (A)
- new net: R20.2, U7.3 (LT), U7.4 (BI), U7.5 (RBI)
- new net: R18.1, U7.14 (g)
- new net: R18.2, U8.3 (G)
- new net: R8.1, U7.11 (c)
- new net: R6.1, U7.12 (b)
- new net: R17.1, U7.15 (f)
- new net: R17.2, U8.2 (F)
- new net: R8.2, U8.8 (C)
- new net: R6.2, U8.9 (B)
- new net: R10.2, U3.10 (J), U3.11 (K)
- new net REST: U3.12 (R), U3.4 (R), U4.12 (R), U5.12 (R)
- no-connect marks 1 -> 6
Other:
- note added: "Montažne rupe"
- note added: "Napajanje bistabila"
- note added: "Reset brojača"
- moved on the sheet: D2, D3, D4, D5, R6, R7, R8, R9, U6
